Commit message: thie robot work

File: simulaitor/robots/robot.urdf (robot description, URDF)
Before this commit: robot square_robot, 2 links, 1 joints
Links:
- added link right_wheel, mass 1; collision cylinder length=0.05 radius=0.1; visual cylinder length=0.05 radius=0.1
Joints:
- added joint right_wheel_joint: type continuous, parent base_link, child right_wheel, origin xyz=0 -0.3 0 rpy=-1.5707 0 0, axis 0 0 1
