Commit message: add robot parts

File: Rover_completo_STL/urfd/stl_test.urdf (robot description, URDF)
Before this commit: robot rover, 2 links, 1 joints
Links:
- added link p2; collision mesh filename=file:///app/stl/Parte2.STL scale=0.01 0.01 0.01; visual mesh filename=file:///app/stl/Parte2.STL scale=0.01 0.01 0.01
- added link p3; collision mesh filename=file:///app/stl/Parte3.STL scale=0.01 0.01 0.01; visual mesh filename=file:///app/stl/Parte3.STL scale=0.01 0.01 0.01
- added link p4; collision mesh filename=file:///app/stl/Parte4.STL scale=0.01 0.01 0.01; visual mesh filename=file:///app/stl/Parte4.STL scale=0.01 0.01 0.01
- added link p5; collision mesh filename=file:///app/stl/Parte5.STL scale=0.01 0.01 0.01; visual mesh filename=file:///app/stl/Parte5.STL scale=0.01 0.01 0.01
- added link p6; collision mesh filename=file:///app/stl/Parte6.STL scale=0.01 0.01 0.01; visual mesh filename=file:///app/stl/Parte6.STL scale=0.01 0.01 0.01
- link base_link: geometry collision mesh filename=file:///app/stl/Parte1.STL scale=0.01 0.01 0.01; visual mesh filename=file:///app/stl/Parte1.STL scale=0.01 0.01 0.01
Joints:
- added joint world_to_base2: type fixed, parent base_link, child p2, origin xyz=0 0 0 rpy=0 0 0
- added joint world_to_base3: type fixed, parent base_link, child p3, origin xyz=0 0 0 rpy=0 0 0
- added joint world_to_base4: type fixed, parent base_link, child p4, origin xyz=0 0 0 rpy=0 0 0
- added joint world_to_base5: type fixed, parent base_link, child p5, origin xyz=0 0 0 rpy=0 0 0
- added joint world_to_base6: type fixed, parent base_link, child p6, origin xyz=0 0 0 rpy=0 0 0
