Commit message: the robot work

File: project/install/base_link_p3_description/share/base_link_p3_description/urdf/base_link_p3.xacro (robot description, xacro)
@@ -2,10 +2,10 @@
 <robot name="base_link_p3" xmlns:xacro="http://www.ros.org/wiki/xacro">
 <xacro:include filename="$(find base_link_p3_description)/urdf/materials.xacro" />
-<xacro:include filename="$(find base_link_p3_description)/urdf/base_link_p3.trans" />
+<xacro:include filename="$(find base_link_p3_description)/urdf/base_link_p3.ros2control" />
 <xacro:include filename="$(find base_link_p3_description)/urdf/base_link_p3.gazebo" />
 <link name="base_link">
   <inertial>
-    <origin xyz="0.4882383881861825 0.14983639102105517 1.1930603195605387" rpy="0 0 0"/>
-    <mass value="46.37689397650178"/>
+    <origin xyz="0.48823838818618254 0.14983639102105534 1.1930603195605385" rpy="0 0 0"/>
+    <mass value="46.376893976501755"/>
     <inertia ixx="2.002069" iyy="3.88283" izz="4.845997" ixy="0.001994" iyz="-0.000599" ixz="0.602482"/>
   </inertial>
@@ -44,5 +44,5 @@
   </collision>
 </link>
-<link name="old_component_1">
+<link name="body_1">
   <inertial>
     <origin xyz="-4.1475883898120514e-05 0.004808803274935047 -0.1762628238361843" rpy="0 0 0"/>
@@ -53,5 +53,5 @@
     <origin xyz="0.049991 -0.517322 -1.133273" rpy="0 0 0"/>
     <geometry>
-      <mesh filename="file://$(find base_link_p3_description)/meshes/old_component_1.stl" scale="0.001 0.001 0.001"/>
+      <mesh filename="file://$(find base_link_p3_description)/meshes/body_1.stl" scale="0.001 0.001 0.001"/>
     </geometry>
     <material name="silver"/>
@@ -60,9 +60,9 @@
     <origin xyz="0.049991 -0.517322 -1.133273" rpy="0 0 0"/>
     <geometry>
-      <mesh filename="file://$(find base_link_p3_description)/meshes/old_component_1.stl" scale="0.001 0.001 0.001"/>
-    </geometry>
-  </collision>
-</link>
-<link name="old_component_3">
+      <mesh filename="file://$(find base_link_p3_description)/meshes/body_1.stl" scale="0.001 0.001 0.001"/>
+    </geometry>
+  </collision>
+</link>
+<link name="body_3">
   <inertial>
     <origin xyz="-4.1461578783374975e-05 0.004808803274935047 -0.1762628238361843" rpy="0 0 0"/>
@@ -73,5 +73,5 @@
     <origin xyz="-0.770009 -0.517322 -1.133273" rpy="0 0 0"/>
     <geometry>
-      <mesh filename="file://$(find base_link_p3_description)/meshes/old_component_3.stl" scale="0.001 0.001 0.001"/>
+      <mesh filename="file://$(find base_link_p3_description)/meshes/body_3.stl" scale="0.001 0.001 0.001"/>
     </geometry>
     <material name="silver"/>
@@ -80,45 +80,45 @@
     <origin xyz="-0.770009 -0.517322 -1.133273" rpy="0 0 0"/>
     <geometry>
-      <mesh filename="file://$(find base_link_p3_description)/meshes/old_component_3.stl" scale="0.001 0.001 0.001"/>
-    </geometry>
-  </collision>
-</link>
-<link name="old_component_4">
-  <inertial>
-    <origin xyz="4.141250651723549e-05 -0.004809646612946972 -0.17626283476147864" rpy="0 0 0"/>
+      <mesh filename="file://$(find base_link_p3_description)/meshes/body_3.stl" scale="0.001 0.001 0.001"/>
+    </geometry>
+  </collision>
+</link>
+<link name="body_4">
+  <inertial>
+    <origin xyz="4.143158000458058e-05 -0.004809645850008343 -0.1762628323772918" rpy="0 0 0"/>
     <mass value="8.196233975814405"/>
     <inertia ixx="0.06724" iyy="0.050751" izz="0.028045" ixy="-2e-05" iyz="-0.006226" ixz="1.4e-05"/>
   </inertial>
   <visual>
-    <origin xyz="-0.769997 0.107318 -1.133279" rpy="0 0 0"/>
-    <geometry>
-      <mesh filename="file://$(find base_link_p3_description)/meshes/old_component_4.stl" scale="0.001 0.001 0.001"/>
-    </geometry>
-    <material name="silver"/>
-  </visual>
-  <collision>
-    <origin xyz="-0.769997 0.107318 -1.133279" rpy="0 0 0"/>
-    <geometry>
-      <mesh filename="file://$(find base_link_p3_description)/meshes/old_component_4.stl" scale="0.001 0.001 0.001"/>
-    </geometry>
-  </collision>
-</link>
-<link name="old_component_5">
-  <inertial>
-    <origin xyz="4.139820140312139e-05 -0.00480964661294761 -0.17626283476147708" rpy="0 0 0"/>
+    <origin xyz="-0.769997 0.110618 -1.133279" rpy="0 0 0"/>
+    <geometry>
+      <mesh filename="file://$(find base_link_p3_description)/meshes/body_4.stl" scale="0.001 0.001 0.001"/>
+    </geometry>
+    <material name="silver"/>
+  </visual>
+  <collision>
+    <origin xyz="-0.769997 0.110618 -1.133279" rpy="0 0 0"/>
+    <geometry>
+      <mesh filename="file://$(find base_link_p3_description)/meshes/body_4.stl" scale="0.001 0.001 0.001"/>
+    </geometry>
+  </collision>
+</link>
+<link name="body_5">
+  <inertial>
+    <origin xyz="4.141727489074404e-05 -0.004809645850008135 -0.17626283237729146" rpy="0 0 0"/>
     <mass value="8.196233975814405"/>
     <inertia ixx="0.06724" iyy="0.050751" izz="0.028045" ixy="-2e-05" iyz="-0.006226" ixz="1.4e-05"/>
   </inertial>
   <visual>
-    <origin xyz="0.050003 0.107318 -1.133279" rpy="0 0 0"/>
-    <geometry>
-      <mesh filename="file://$(find base_link_p3_description)/meshes/old_component_5.stl" scale="0.001 0.001 0.001"/>
-    </geometry>
-    <material name="silver"/>
-  </visual>
-  <collision>
-    <origin xyz="0.050003 0.107318 -1.133279" rpy="0 0 0"/>
-    <geometry>
-      <mesh filename="file://$(find base_link_p3_description)/meshes/old_component_5.stl" scale="0.001 0.001 0.001"/>
+    <origin xyz="0.050003 0.110618 -1.133279" rpy="0 0 0"/>
+    <geometry>
+      <mesh filename="file://$(find base_link_p3_description)/meshes/body_5.stl" scale="0.001 0.001 0.001"/>
+    </geometry>
+    <material name="silver"/>
+  </visual>
+  <collision>
+    <origin xyz="0.050003 0.110618 -1.133279" rpy="0 0 0"/>
+    <geometry>
+      <mesh filename="file://$(find base_link_p3_description)/meshes/body_5.stl" scale="0.001 0.001 0.001"/>
     </geometry>
   </collision>
@@ -126,5 +126,5 @@
 <link name="Parte1__17__2">
   <inertial>
-    <origin xyz="0.0007132805534282305 0.0596212723884173 -0.024439230247864208" rpy="0 0 0"/>
+    <origin xyz="0.0007132996269144654 0.056321273151356654 -0.024439227863678914" rpy="0 0 0"/>
     <mass value="11.344297541309349"/>
     <inertia ixx="0.034487" iyy="1.409892" izz="1.396504" ixy="0.000254" iyz="-0.003774" ixz="-0.000343"/>
@@ -146,7 +146,7 @@
 <link name="Parte6_2">
   <inertial>
-    <origin xyz="-0.0004342840487971955 -0.07079622839421573 -0.000331842682977479" rpy="0 0 0"/>
-    <mass value="18.53573494070931"/>
-    <inertia ixx="0.086336" iyy="0.143083" izz="0.086786" ixy="0.000124" iyz="8.1e-05" ixz="-0.000509"/>
+    <origin xyz="-0.0009038326245139894 -0.055001544958308 -0.0006381400064267018" rpy="0 0 0"/>
+    <mass value="8.776606415040463"/>
+    <inertia ixx="0.060833" iyy="0.104458" izz="0.061281" ixy="0.0" iyz="0.0" ixz="-0.000507"/>
   </inertial>
   <visual>
@@ -166,10 +166,10 @@
 <link name="Parte6_4">
   <inertial>
-    <origin xyz="-0.0028636125080598387 0.039203598028237696 -0.004274720976729873" rpy="0 0 0"/>
-    <mass value="18.53573494070931"/>
-    <inertia ixx="0.086336" iyy="0.143083" izz="0.086786" ixy="0.000124" iyz="8.1e-05" ixz="-0.000509"/>
-  </inertial>
-  <visual>
-    <origin xyz="0.049991 0.241315 -0.908279" rpy="0 0 0"/>
+    <origin xyz="-0.0033331420102889267 0.05499828222708522 -0.004581015915993025" rpy="0 0 0"/>
+    <mass value="8.776606415040463"/>
+    <inertia ixx="0.060833" iyy="0.104458" izz="0.061281" ixy="0.0" iyz="0.0" ixz="-0.000507"/>
+  </inertial>
+  <visual>
+    <origin xyz="0.049991 0.244615 -0.908279" rpy="0 0 0"/>
     <geometry>
       <mesh filename="file://$(find base_link_p3_description)/meshes/Parte6_4.stl" scale="0.001 0.001 0.001"/>
@@ -178,5 +178,5 @@
   </visual>
   <collision>
-    <origin xyz="0.049991 0.241315 -0.908279" rpy="0 0 0"/>
+    <origin xyz="0.049991 0.244615 -0.908279" rpy="0 0 0"/>
     <geometry>
       <mesh filename="file://$(find base_link_p3_description)/meshes/Parte6_4.stl" scale="0.001 0.001 0.001"/>
@@ -186,10 +186,10 @@
 <link name="Parte6_5">
   <inertial>
-    <origin xyz="0.0004341191470640382 0.07079557856816679 -0.0003318726817584938" rpy="0 0 0"/>
-    <mass value="18.53573494070931"/>
-    <inertia ixx="0.086336" iyy="0.143083" izz="0.086786" ixy="0.000124" iyz="-8.1e-05" ixz="0.000509"/>
-  </inertial>
-  <visual>
-    <origin xyz="-0.770009 0.241315 -0.908279" rpy="0 0 0"/>
+    <origin xyz="0.0009036867962681772 0.05500089589519774 -0.0006381676210214238" rpy="0 0 0"/>
+    <mass value="8.776606415040463"/>
+    <inertia ixx="0.060833" iyy="0.104458" izz="0.061281" ixy="0.0" iyz="-0.0" ixz="0.000507"/>
+  </inertial>
+  <visual>
+    <origin xyz="-0.770009 0.244615 -0.908279" rpy="0 0 0"/>
     <geometry>
       <mesh filename="file://$(find base_link_p3_description)/meshes/Parte6_5.stl" scale="0.001 0.001 0.001"/>
@@ -198,5 +198,5 @@
   </visual>
   <collision>
-    <origin xyz="-0.770009 0.241315 -0.908279" rpy="0 0 0"/>
+    <origin xyz="-0.770009 0.244615 -0.908279" rpy="0 0 0"/>
     <geometry>
       <mesh filename="file://$(find base_link_p3_description)/meshes/Parte6_5.stl" scale="0.001 0.001 0.001"/>
@@ -206,7 +206,7 @@
 <link name="Parte6_3">
   <inertial>
-    <origin xyz="0.00042233138036879697 0.010795558633750146 -0.0002757643979985902" rpy="0 0 0"/>
-    <mass value="18.53573494070931"/>
-    <inertia ixx="0.086336" iyy="0.143083" izz="0.086786" ixy="0.000124" iyz="-8.1e-05" ixz="0.000509"/>
+    <origin xyz="-0.0033329675718140744 0.05499826316885659 -0.004581007374887314" rpy="0 0 0"/>
+    <mass value="8.776606415040463"/>
+    <inertia ixx="0.060833" iyy="0.104458" izz="0.061281" ixy="0.0" iyz="0.0" ixz="-0.000507"/>
   </inertial>
   <visual>
@@ -224,13 +224,14 @@
   </collision>
 </link>
-<joint name="R�gido 2" type="fixed">
+<joint name="Revolucionar 2" type="continuous">
   <origin xyz="0.360009 0.49 1.192273" rpy="0 0 0"/>
   <parent link="base_link"/>
   <child link="Parte1__17__1"/>
+  <axis xyz="0.0 1.0 0.0"/>
 </joint>
 <joint name="Revolucionar 3" type="continuous">
   <origin xyz="-0.41 0.027322 -0.059" rpy="0 0 0"/>
   <parent link="Parte1__17__1"/>
-  <child link="old_component_1"/>
+  <child link="body_1"/>
   <axis xyz="0.0 0.0 -1.0"/>
 </joint>
@@ -238,27 +239,28 @@
   <origin xyz="0.41 0.027322 -0.059" rpy="0 0 0"/>
   <parent link="Parte1__17__1"/>
-  <child link="old_component_3"/>
+  <child link="body_3"/>
   <axis xyz="0.0 0.0 -1.0"/>
 </joint>
 <joint name="Revolucionar 5" type="continuous">
-  <origin xyz="0.41 0.082682 -0.059" rpy="0 0 0"/>
+  <origin xyz="0.41 0.079382 -0.059" rpy="0 0 0"/>
   <parent link="Parte1__17__2"/>
-  <child link="old_component_4"/>
+  <child link="body_4"/>
   <axis xyz="-0.0 0.0 -1.0"/>
 </joint>
 <joint name="Revolucionar 6" type="continuous">
-  <origin xyz="-0.41 0.082682 -0.059" rpy="0 0 0"/>
+  <origin xyz="-0.41 0.079382 -0.059" rpy="0 0 0"/>
   <parent link="Parte1__17__2"/>
-  <child link="old_component_5"/>
+  <child link="body_5"/>
   <axis xyz="-0.0 0.0 -1.0"/>
 </joint>
-<joint name="R�gido 7" type="fixed">
+<joint name="Revolucionar 7" type="continuous">
   <origin xyz="0.359997 -0.19 1.192279" rpy="0 0 0"/>
   <parent link="base_link"/>
   <child link="Parte1__17__2"/>
+  <axis xyz="0.0 -1.0 0.0"/>
 </joint>
 <joint name="Revolucionar 8" type="continuous">
   <origin xyz="-6e-06 0.122735 -0.225" rpy="0 0 0"/>
-  <parent link="old_component_3"/>
+  <parent link="body_3"/>
   <child link="Parte6_2"/>
   <axis xyz="0.0 1.0 0.0"/>
@@ -266,11 +268,11 @@
 <joint name="Revolucionar 10" type="continuous">
   <origin xyz="1.2e-05 -0.133997 -0.225" rpy="0 0 0"/>
-  <parent link="old_component_5"/>
+  <parent link="body_5"/>
   <child link="Parte6_4"/>
-  <axis xyz="0.0 -1.0 -0.0"/>
+  <axis xyz="-0.0 -1.0 0.0"/>
 </joint>
 <joint name="Revolucionar 11" type="continuous">
   <origin xyz="1.2e-05 -0.133997 -0.225" rpy="0 0 0"/>
-  <parent link="old_component_4"/>
+  <parent link="body_4"/>
   <child link="Parte6_5"/>
   <axis xyz="0.0 -1.0 -0.0"/>
@@ -278,5 +280,5 @@
 <joint name="Revolucionar 12" type="continuous">
   <origin xyz="-1.2e-05 0.133997 -0.225" rpy="0 0 0"/>
-  <parent link="old_component_1"/>
+  <parent link="body_1"/>
   <child link="Parte6_3"/>
   <axis xyz="0.0 1.0 0.0"/>

Commit message: start config gazebo contorlers

File: project/install/base_link_p3_description/share/base_link_p3_description/urdf/base_link_p3.xacro (robot description, xacro)
@@ -254,5 +254,5 @@
   <axis xyz="-0.0 0.0 -1.0"/>
 </joint>
-<joint name="Revolucionar 7" type="continuous">
+<joint name="revolucionar_7" type="continuous">
   <origin xyz="0.359997 -0.19 1.192279" rpy="0 0 0"/>
   <parent link="base_link"/>

Commit message: update dirver the robot

File: project/install/base_link_p3_description/share/base_link_p3_description/urdf/base_link_p3.xacro (robot description, xacro)
@@ -224,5 +224,5 @@
   </collision>
 </link>
-<joint name="Revolucionar 2" type="continuous">
+<joint name="revolucionar_2" type="continuous">
   <origin xyz="0.360009 0.49 1.192273" rpy="0 0 0"/>
   <parent link="base_link"/>
@@ -230,5 +230,5 @@
   <axis xyz="0.0 1.0 0.0"/>
 </joint>
-<joint name="Revolucionar 3" type="continuous">
+<joint name="revolucionar_3" type="continuous">
   <origin xyz="-0.41 0.027322 -0.059" rpy="0 0 0"/>
   <parent link="Parte1__17__1"/>
@@ -236,5 +236,5 @@
   <axis xyz="0.0 0.0 -1.0"/>
 </joint>
-<joint name="Revolucionar 4" type="continuous">
+<joint name="revolucionar_4" type="continuous">
   <origin xyz="0.41 0.027322 -0.059" rpy="0 0 0"/>
   <parent link="Parte1__17__1"/>
@@ -242,5 +242,5 @@
   <axis xyz="0.0 0.0 -1.0"/>
 </joint>
-<joint name="Revolucionar 5" type="continuous">
+<joint name="revolucionar_5" type="continuous">
   <origin xyz="0.41 0.079382 -0.059" rpy="0 0 0"/>
   <parent link="Parte1__17__2"/>
@@ -248,5 +248,5 @@
   <axis xyz="-0.0 0.0 -1.0"/>
 </joint>
-<joint name="Revolucionar 6" type="continuous">
+<joint name="revolucionar_6" type="continuous">
   <origin xyz="-0.41 0.079382 -0.059" rpy="0 0 0"/>
   <parent link="Parte1__17__2"/>
@@ -260,5 +260,5 @@
   <axis xyz="0.0 -1.0 0.0"/>
 </joint>
-<joint name="Revolucionar 8" type="continuous">
+<joint name="revolucionar_8" type="continuous">
   <origin xyz="-6e-06 0.122735 -0.225" rpy="0 0 0"/>
   <parent link="body_3"/>
@@ -266,5 +266,5 @@
   <axis xyz="0.0 1.0 0.0"/>
 </joint>
-<joint name="Revolucionar 10" type="continuous">
+<joint name="revolucionar_10" type="continuous">
   <origin xyz="1.2e-05 -0.133997 -0.225" rpy="0 0 0"/>
   <parent link="body_5"/>
@@ -272,5 +272,5 @@
   <axis xyz="-0.0 -1.0 0.0"/>
 </joint>
-<joint name="Revolucionar 11" type="continuous">
+<joint name="revolucionar_11" type="continuous">
   <origin xyz="1.2e-05 -0.133997 -0.225" rpy="0 0 0"/>
   <parent link="body_4"/>
@@ -278,5 +278,5 @@
   <axis xyz="0.0 -1.0 -0.0"/>
 </joint>
-<joint name="Revolucionar 12" type="continuous">
+<joint name="revolucionar_12" type="continuous">
   <origin xyz="-1.2e-05 0.133997 -0.225" rpy="0 0 0"/>
   <parent link="body_1"/>
