Commit message: chage name robot

File: project/src/bart/urdf/bart.urdf (robot description, URDF)
Before this commit: robot base_link_p3, 11 links, 10 joints
Links:
- link Parte1__17__1: geometry collision mesh filename=file://$(find bart)/meshes/Parte1__17__1.stl scale=0.001 0.001 0.001; visual mesh filename=file://$(find bart)/meshes/Parte1__17__1.stl scale=0.001 0.001 0.001
- link Parte1__17__2: geometry collision mesh filename=file://$(find bart)/meshes/Parte1__17__2.stl scale=0.001 0.001 0.001; visual mesh filename=file://$(find bart)/meshes/Parte1__17__2.stl scale=0.001 0.001 0.001
- link Parte6_2: geometry collision mesh filename=file://$(find bart)/meshes/Parte6_2.stl scale=0.001 0.001 0.001; visual mesh filename=file://$(find bart)/meshes/Parte6_2.stl scale=0.001 0.001 0.001
- link Parte6_3: geometry collision mesh filename=file://$(find bart)/meshes/Parte6_3.stl scale=0.001 0.001 0.001; visual mesh filename=file://$(find bart)/meshes/Parte6_3.stl scale=0.001 0.001 0.001
- link Parte6_4: geometry collision mesh filename=file://$(find bart)/meshes/Parte6_4.stl scale=0.001 0.001 0.001; visual mesh filename=file://$(find bart)/meshes/Parte6_4.stl scale=0.001 0.001 0.001
- link Parte6_5: geometry collision mesh filename=file://$(find bart)/meshes/Parte6_5.stl scale=0.001 0.001 0.001; visual mesh filename=file://$(find bart)/meshes/Parte6_5.stl scale=0.001 0.001 0.001
- link base_link: geometry collision mesh filename=file://$(find bart)/meshes/base_link.stl scale=0.001 0.001 0.001; visual mesh filename=file://$(find bart)/meshes/base_link.stl scale=0.001 0.001 0.001
- link old_component_1: geometry collision mesh filename=file://$(find bart)/meshes/old_component_1.stl scale=0.001 0.001 0.001; visual mesh filename=file://$(find bart)/meshes/old_component_1.stl scale=0.001 0.001 0.001
- link old_component_3: geometry collision mesh filename=file://$(find bart)/meshes/old_component_3.stl scale=0.001 0.001 0.001; visual mesh filename=file://$(find bart)/meshes/old_component_3.stl scale=0.001 0.001 0.001
- link old_component_4: geometry collision mesh filename=file://$(find bart)/meshes/old_component_4.stl scale=0.001 0.001 0.001; visual mesh filename=file://$(find bart)/meshes/old_component_4.stl scale=0.001 0.001 0.001
- link old_component_5: geometry collision mesh filename=file://$(find bart)/meshes/old_component_5.stl scale=0.001 0.001 0.001; visual mesh filename=file://$(find bart)/meshes/old_component_5.stl scale=0.001 0.001 0.001

File: project/src/bart/urdf/bart.xacro (robot description, xacro)
@@ -1,7 +1,7 @@
 <?xml version="1.0" ?>
-<robot name="base_link_p3" xmlns:xacro="http://www.ros.org/wiki/xacro">
-<xacro:include filename="$(find base_link_p3_description)/urdf/materials.xacro" />
-<xacro:include filename="$(find base_link_p3_description)/urdf/base_link_p3.ros2control" />
-<xacro:include filename="$(find base_link_p3_description)/urdf/base_link_p3.gazebo" />
+<robot name="bart" xmlns:xacro="http://www.ros.org/wiki/xacro">
+<xacro:include filename="$(find bart)/urdf/materials.xacro" />
+<xacro:include filename="$(find bart)/urdf/bart.ros2control" />
+<xacro:include filename="$(find bart)/urdf/bart.gazebo" />
 <link name="base_link">
   <inertial>
@@ -13,5 +13,5 @@
     <origin xyz="0 0 0" rpy="0 0 0"/>
     <geometry>
-      <mesh filename="file://$(find base_link_p3_description)/meshes/base_link.stl" scale="0.001 0.001 0.001"/>
+      <mesh filename="file://$(find bart)/meshes/base_link.stl" scale="0.001 0.001 0.001"/>
     </geometry>
     <material name="silver"/>
@@ -20,5 +20,5 @@
     <origin xyz="0 0 0" rpy="0 0 0"/>
     <geometry>
-      <mesh filename="file://$(find base_link_p3_description)/meshes/base_link.stl" scale="0.001 0.001 0.001"/>
+      <mesh filename="file://$(find bart)/meshes/base_link.stl" scale="0.001 0.001 0.001"/>
     </geometry>
   </collision>
@@ -33,5 +33,5 @@
     <origin xyz="-0.360009 -0.49 -1.192273" rpy="0 0 0"/>
     <geometry>
-      <mesh filename="file://$(find base_link_p3_description)/meshes/Parte1__17__1.stl" scale="0.001 0.001 0.001"/>
+      <mesh filename="file://$(find bart)/meshes/Parte1__17__1.stl" scale="0.001 0.001 0.001"/>
     </geometry>
     <material name="silver"/>
@@ -40,5 +40,5 @@
     <origin xyz="-0.360009 -0.49 -1.192273" rpy="0 0 0"/>
     <geometry>
-      <mesh filename="file://$(find base_link_p3_description)/meshes/Parte1__17__1.stl" scale="0.001 0.001 0.001"/>
+      <mesh filename="file://$(find bart)/meshes/Parte1__17__1.stl" scale="0.001 0.001 0.001"/>
     </geometry>
   </collision>
@@ -53,5 +53,5 @@
     <origin xyz="0.049991 -0.517322 -1.133273" rpy="0 0 0"/>
     <geometry>
-      <mesh filename="file://$(find base_link_p3_description)/meshes/body_1.stl" scale="0.001 0.001 0.001"/>
+      <mesh filename="file://$(find bart)/meshes/body_1.stl" scale="0.001 0.001 0.001"/>
     </geometry>
     <material name="silver"/>
@@ -60,5 +60,5 @@
     <origin xyz="0.049991 -0.517322 -1.133273" rpy="0 0 0"/>
     <geometry>
-      <mesh filename="file://$(find base_link_p3_description)/meshes/body_1.stl" scale="0.001 0.001 0.001"/>
+      <mesh filename="file://$(find bart)/meshes/body_1.stl" scale="0.001 0.001 0.001"/>
     </geometry>
   </collision>
@@ -73,5 +73,5 @@
     <origin xyz="-0.770009 -0.517322 -1.133273" rpy="0 0 0"/>
     <geometry>
-      <mesh filename="file://$(find base_link_p3_description)/meshes/body_3.stl" scale="0.001 0.001 0.001"/>
+      <mesh filename="file://$(find bart)/meshes/body_3.stl" scale="0.001 0.001 0.001"/>
     </geometry>
     <material name="silver"/>
@@ -80,5 +80,5 @@
     <origin xyz="-0.770009 -0.517322 -1.133273" rpy="0 0 0"/>
     <geometry>
-      <mesh filename="file://$(find base_link_p3_description)/meshes/body_3.stl" scale="0.001 0.001 0.001"/>
+      <mesh filename="file://$(find bart)/meshes/body_3.stl" scale="0.001 0.001 0.001"/>
     </geometry>
   </collision>
@@ -93,5 +93,5 @@
     <origin xyz="-0.769997 0.110618 -1.133279" rpy="0 0 0"/>
     <geometry>
-      <mesh filename="file://$(find base_link_p3_description)/meshes/body_4.stl" scale="0.001 0.001 0.001"/>
+      <mesh filename="file://$(find bart)/meshes/body_4.stl" scale="0.001 0.001 0.001"/>
     </geometry>
     <material name="silver"/>
@@ -100,5 +100,5 @@
     <origin xyz="-0.769997 0.110618 -1.133279" rpy="0 0 0"/>
     <geometry>
-      <mesh filename="file://$(find base_link_p3_description)/meshes/body_4.stl" scale="0.001 0.001 0.001"/>
+      <mesh filename="file://$(find bart)/meshes/body_4.stl" scale="0.001 0.001 0.001"/>
     </geometry>
   </collision>
@@ -113,5 +113,5 @@
     <origin xyz="0.050003 0.110618 -1.133279" rpy="0 0 0"/>
     <geometry>
-      <mesh filename="file://$(find base_link_p3_description)/meshes/body_5.stl" scale="0.001 0.001 0.001"/>
+      <mesh filename="file://$(find bart)/meshes/body_5.stl" scale="0.001 0.001 0.001"/>
     </geometry>
     <material name="silver"/>
@@ -120,5 +120,5 @@
     <origin xyz="0.050003 0.110618 -1.133279" rpy="0 0 0"/>
     <geometry>
-      <mesh filename="file://$(find base_link_p3_description)/meshes/body_5.stl" scale="0.001 0.001 0.001"/>
+      <mesh filename="file://$(find bart)/meshes/body_5.stl" scale="0.001 0.001 0.001"/>
     </geometry>
   </collision>
@@ -133,5 +133,5 @@
     <origin xyz="-0.359997 0.19 -1.192279" rpy="0 0 0"/>
     <geometry>
-      <mesh filename="file://$(find base_link_p3_description)/meshes/Parte1__17__2.stl" scale="0.001 0.001 0.001"/>
+      <mesh filename="file://$(find bart)/meshes/Parte1__17__2.stl" scale="0.001 0.001 0.001"/>
     </geometry>
     <material name="silver"/>
@@ -140,5 +140,5 @@
     <origin xyz="-0.359997 0.19 -1.192279" rpy="0 0 0"/>
     <geometry>
-      <mesh filename="file://$(find base_link_p3_description)/meshes/Parte1__17__2.stl" scale="0.001 0.001 0.001"/>
+      <mesh filename="file://$(find bart)/meshes/Parte1__17__2.stl" scale="0.001 0.001 0.001"/>
     </geometry>
   </collision>
@@ -153,5 +153,5 @@
     <origin xyz="-0.770003 -0.640057 -0.908273" rpy="0 0 0"/>
     <geometry>
-      <mesh filename="file://$(find base_link_p3_description)/meshes/Parte6_2.stl" scale="0.001 0.001 0.001"/>
+      <mesh filename="file://$(find bart)/meshes/Parte6_2.stl" scale="0.001 0.001 0.001"/>
     </geometry>
     <material name="silver"/>
@@ -160,5 +160,5 @@
     <origin xyz="-0.770003 -0.640057 -0.908273" rpy="0 0 0"/>
     <geometry>
-      <mesh filename="file://$(find base_link_p3_description)/meshes/Parte6_2.stl" scale="0.001 0.001 0.001"/>
+      <mesh filename="file://$(find bart)/meshes/Parte6_2.stl" scale="0.001 0.001 0.001"/>
     </geometry>
   </collision>
@@ -173,5 +173,5 @@
     <origin xyz="0.049991 0.244615 -0.908279" rpy="0 0 0"/>
     <geometry>
-      <mesh filename="file://$(find base_link_p3_description)/meshes/Parte6_4.stl" scale="0.001 0.001 0.001"/>
+      <mesh filename="file://$(find bart)/meshes/Parte6_4.stl" scale="0.001 0.001 0.001"/>
     </geometry>
     <material name="silver"/>
@@ -180,5 +180,5 @@
     <origin xyz="0.049991 0.244615 -0.908279" rpy="0 0 0"/>
     <geometry>
-      <mesh filename="file://$(find base_link_p3_description)/meshes/Parte6_4.stl" scale="0.001 0.001 0.001"/>
+      <mesh filename="file://$(find bart)/meshes/Parte6_4.stl" scale="0.001 0.001 0.001"/>
     </geometry>
   </collision>
@@ -193,5 +193,5 @@
     <origin xyz="-0.770009 0.244615 -0.908279" rpy="0 0 0"/>
     <geometry>
-      <mesh filename="file://$(find base_link_p3_description)/meshes/Parte6_5.stl" scale="0.001 0.001 0.001"/>
+      <mesh filename="file://$(find bart)/meshes/Parte6_5.stl" scale="0.001 0.001 0.001"/>
     </geometry>
     <material name="silver"/>
@@ -200,5 +200,5 @@
     <origin xyz="-0.770009 0.244615 -0.908279" rpy="0 0 0"/>
     <geometry>
-      <mesh filename="file://$(find base_link_p3_description)/meshes/Parte6_5.stl" scale="0.001 0.001 0.001"/>
+      <mesh filename="file://$(find bart)/meshes/Parte6_5.stl" scale="0.001 0.001 0.001"/>
     </geometry>
   </collision>
@@ -213,5 +213,5 @@
     <origin xyz="0.050003 -0.651319 -0.908273" rpy="0 0 0"/>
     <geometry>
-      <mesh filename="file://$(find base_link_p3_description)/meshes/Parte6_3.stl" scale="0.001 0.001 0.001"/>
+      <mesh filename="file://$(find bart)/meshes/Parte6_3.stl" scale="0.001 0.001 0.001"/>
     </geometry>
     <material name="silver"/>
@@ -220,5 +220,5 @@
     <origin xyz="0.050003 -0.651319 -0.908273" rpy="0 0 0"/>
     <geometry>
-      <mesh filename="file://$(find base_link_p3_description)/meshes/Parte6_3.stl" scale="0.001 0.001 0.001"/>
+      <mesh filename="file://$(find bart)/meshes/Parte6_3.stl" scale="0.001 0.001 0.001"/>
     </geometry>
   </collision>

File: project/src/bart/urdf/materials.xacro (robot description, xacro)
@@ -1,4 +1,4 @@
 <?xml version="1.0" ?>
-<robot name="base_link_p3" xmlns:xacro="http://www.ros.org/wiki/xacro" >
+<robot name="bart" xmlns:xacro="http://www.ros.org/wiki/xacro" >
 <material name="silver">
   <color rgba="0.700 0.700 0.700 1.000"/>
