Commit message: Fix LiDAR sensor configuration with proper topic and gz_ros2_control plugin

File: project/src/bart/urdf/lidar.xacro (robot description, xacro)
@@ -28,3 +28,34 @@
     <child link="lidar_1"/>
   </joint>
+  <!-- LiDAR Gazebo plugin configuration -->
+  <gazebo reference="lidar_1">
+    <material>Gazebo/Black</material>
+    <sensor name="lidar_sensor" type="gpu_lidar">
+      <topic>lidar_1/scan</topic>
+      <update_rate>10</update_rate>
+      <ray>
+        <scan>
+          <horizontal>
+            <samples>360</samples>
+            <resolution>1</resolution>
+            <min_angle>-3.14159265359</min_angle>
+            <max_angle>3.14159265359</max_angle>
+          </horizontal>
+          <vertical>
+            <samples>16</samples>
+            <resolution>1</resolution>
+            <min_angle>-0.261799</min_angle>
+            <max_angle>0.261799</max_angle>
+          </vertical>
+        </scan>
+        <range>
+          <min>0.08</min>
+          <max>30.0</max>
+          <resolution>0.01</resolution>
+        </range>
+      </ray>
+      <always_on>true</always_on>
+      <visualize>true</visualize>
+    </sensor>
+  </gazebo>
 </robot>

Commit message: upadte lidar location

File: project/src/bart/urdf/lidar.xacro (robot description, xacro)
@@ -25,12 +25,12 @@
     <parent link="base_link" />
     <child link="lidar_link" />
-    <origin xyz="0 0 0.2" rpy="0 0 0" />
+    <origin xyz="0 0 1.5" rpy="0 0 0" />
   </joint>
   <gazebo reference="lidar_link">
     <sensor name="lidar" type="gpu_lidar">
+      <visualize>true</visualize>
       <pose>0 0 0 0 0 0</pose>
       <update_rate>10</update_rate>
       <always_on>true</always_on>
-      <visualize>true</visualize>
       <ray>
         <scan>
